File: asserv_shield/shield/motor_shield.brd (EAGLE design)
At the start: 100 x 100 mm, 83 parts, among them IC1 L298, IC2 L298

Commit message: minor updates
Parts:
- removed Q1, Q10, Q11, Q12, Q13, Q14, Q15, Q16, Q17, Q18, Q19, Q2, Q20, Q25, Q26, Q27, Q28, Q3, Q4, Q9: (no value), semicon-smd-ipc:SOT23
- removed R10, R20, R22, R24, R26, R28, R30, R32, R34, R36, R38, R40, R42, R52, R54, R56, R58, R6, R8: 800, rcl:M0805
- added C1: (no value), BeagleBone_Blue:SPARKFUN-CAPACITORS_0805
- added C2, C3, C4, C5, C6: (no value), BeagleBone_Blue:ADAFRUIT_140CLH-1010
- added IC10, IC11, IC7, IC8, IC9: 74LS19D, 74xx-eu:SO14
- added IC3: 4030D, 40xx:SO14
- added IC4: 7805DT, linear:TO252
- added IC5: MAX6520, maxim:SOT23
- added IC6: LM358D, linear:SO08
- added J10: (no value), SparkFun-Connectors:SCREWTERMINAL-3.5MM-8
- added J11: (no value), con-jack:SPC4078
- added J12: (no value), SparkFun-Connectors:MOLEX-1X2_LOCK
- added K1: RT33K012, relay:RT-N/O16A5
- added Q5, Q6: STRAWSON_EAGLE_LIB_MOSFET-NCHANNEL, BeagleBone_Blue:STRAWSON_EAGLE_LIB_SO08-TIGHT
- added R11: 6k, rcl:M0805
- added R12: 3k, rcl:M0805
- added RN1: (no value), resistor-net:RN-8
- added RN2, RN3, RN4, RN5, RN6: 680, resistor-net:RN-5
- added U$5: XL6009, beffroyables:XL6009
- added X2, X3: (no value), con-phoenix-500:MSTBV2
- R4: value 800 -> 6k
- moved X1 94.0 mm to (96.5, 71.1), turned to 270 degrees
- moved R25 43.7 mm to (51.1, 14.6)
- moved OPT_MOT1 43.0 mm to (58.4, 17.8)
- moved R23 42.7 mm to (51.1, 18.4)
- moved R21 41.7 mm to (51.1, 22.2)
- moved R19 40.4 mm to (51.1, 26.0)
- moved R27 38.8 mm to (70.5, 74.6)
- moved R4 38.7 mm to (53.5, 76.9), turned to 180 degrees
- moved R29 38.2 mm to (70.5, 71.4)
- moved R31 37.1 mm to (70.5, 67.6)
- moved OPT_MISC 36.7 mm to (76.8, 67.6)
- moved R33 36.3 mm to (70.5, 64.5)
- moved U$2 29.2 mm to (31.8, 15.2)
- moved J2 24.4 mm to (25.4, 38.1)
- moved J6 24.4 mm to (33.0, 38.1)
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Connections:
- removed net EN2A: PCB1.P8.35
- removed net MOT_DIR1A: PCB1.P9.28
- removed net MOT_PMW_1B: PCB1.P9.16
- removed net VCC: IC1.9, IC2.9
- new net +12V_PWR: C2.+, C3.+, C4.+, C5.+, IC1.4, IC2.4, J11.3, U$5.IN+, X1.2
- new net +4.1V: U$4.P$10, U$4.P$11, U$4.P$12, U$4.P$21, U$4.P$22, U$4.P$7, U$4.P$8, U$4.P$9, U$5.OUT+
- new net COL1: J10.5, PCB1.P8.4, RN1.5
- new net COL2: J10.4, PCB1.P8.5, RN1.4
- new net DOOR_MOT_1A: IC3.3, OPT_MOT1.2
- new net DOOR_MOT_2A: IC3.4, OPT_MOT1.6
- new net DOOR_MOT_3A: IC3.10, OPT_MOT2.2
- new net DOOR_MOT_4A: IC3.11, OPT_MOT2.6
- new net GREEN: J10.8, PCB1.P8.8, RN1.8
- new net MOT_PWM_1B: IC3.5, PCB1.P9.16
- new net N$64: IC5.2, IC6.2
- new net N$73: IC6.1, R4.2
- new net N$74: K1.14A, K1.14B, X2.2, X3.1
- new net N$75: K1.A1, Q6.5, Q6.6, Q6.7, Q6.8
- new net N$76: IC6.3, J12.2, R11.1, R12.2
- new net N$77: C1.1, Q6.4, R4.1
- new net ORANGE: J10.7, PCB1.P8.7, RN1.7
- new net RED: J10.6, PCB1.P8.6, RN1.6
- new net STOP: J10.3, PCB1.P8.3, RN1.3
- new net TIRETTE: J10.2, PCB1.P8.14, RN1.2
- net +12V: now also IC4.1, K1.11A, K1.11B, K1.A2, R11.2, X1.1, X2.1; no longer IC1.4, IC2.4, X1.2
- net +3V3: now also RN1.1
- net +5V: now also IC1.9, IC10.14, IC11.14, IC2.9, IC4.2, IC5.1, IC6.8, IC7.14, IC8.14, IC9.14, RN2.1, RN3.1, RN4.1, RN5.1, RN6.1; no longer R10.2, R20.2, R22.2, R24.2, R26.2, R28.2, R30.2, R32.2, R34.2, R36.2, R38.2, R4.2, R40.2, R42.2, R52.2, R54.2, R56.2, R58.2, R6.2, R8.2
- net ENC_2A: now also PCB1.P8.35
- net GND: now also C1.2, C2.-, C3.-, C4.-, C5.-, IC10.7, IC11.7, IC4.3, IC5.3, IC6.4, IC7.7, IC8.7, IC9.7, J12.1, Q5.1, Q5.2, Q5.3, Q6.1, Q6.2, Q6.3, R12.1, U$5.IN-, U$5.OUT-, X3.2; no longer OPT_MISC.9, Q1.2, Q10.2, Q11.2, Q12.2, Q13.2, Q14.2, Q15.2, Q16.2, Q17.2, Q18.2, Q19.2, Q2.2, Q20.2, Q25.2, Q26.2, Q27.2, Q28.2, Q3.2, Q4.2, Q9.2, X1.1
- net I2C2_SCL: no longer J9.1
- net I2C2_SDA: now also J9.1
- net MOT_1A: now also IC3.2, PCB1.P9.28; no longer OPT_MOT1.2
- net MOT_2A: now also IC3.6; no longer OPT_MOT1.6
- net MOT_3A: now also IC3.9; no longer OPT_MOT2.2
- net MOT_4A: now also IC3.13; no longer OPT_MOT2.6
- net MOT_PWM_1A: now also IC3.1
- net MOT_PWM_2A: now also IC3.8
- net MOT_PWM_2B: now also IC3.12
- net N$10: now also J11.1, Q5.5, Q5.6, Q5.7, Q5.8; no longer U$4.P$10, U$4.P$11, U$4.P$12, U$4.P$21, U$4.P$22, U$4.P$7, U$4.P$8, U$4.P$9
- net N$19: now also IC9.1, RN4.5; no longer Q4.1
- net N$20: now also IC8.1, RN3.5; no longer Q12.1
- net N$21: now also IC8.9, RN3.4; no longer Q11.1
- net N$30: now also IC8.11, RN3.3; no longer Q10.1
- net N$31: now also IC8.13, RN3.2; no longer Q9.1
- net N$32: now also IC9.13, RN4.2; no longer Q1.1
- net N$33: now also IC9.11, RN4.3; no longer Q2.1
- net N$34: now also IC9.9, RN4.4; no longer Q3.1
- net N$35: now also IC10.1, RN6.5; no longer Q20.1
- net N$36: now also IC10.9, RN6.4; no longer Q19.1
- net N$37: now also IC10.11, RN6.3; no longer Q18.1
- net N$4: now also IC7.13, RN2.2; no longer Q13.1
- net N$46: now also IC10.13, RN6.2; no longer Q17.1
- net N$47: now also IC11.13, RN5.2; no longer Q25.1
- net N$48: now also IC11.11, RN5.3; no longer Q26.1
- net N$49: now also IC11.9, RN5.4; no longer Q27.1
- net N$50: now also IC11.1, RN5.5; no longer Q28.1
- net N$53: now also IC7.11, RN2.3; no longer Q14.1
- net N$62: now also IC7.9, RN2.4; no longer Q15.1
- net N$63: now also IC7.1, RN2.5; no longer Q16.1
- net OPT_MOT1A: now also IC8.12; no longer Q9.3, R20.1
- net OPT_MOT1B: now also IC8.10; no longer Q10.3, R22.1
- net OPT_MOT2A: now also IC8.8; no longer Q11.3, R24.1
- net OPT_MOT2B: now also IC8.2; no longer Q12.3, R26.1
- net OPT_MOT3A: now also IC9.12; no longer Q1.3, R4.1
- net OPT_MOT3B: now also IC9.10; no longer Q2.3, R6.1
- net OPT_MOT4A: now also IC9.8; no longer Q3.3, R8.1
- net OPT_MOT4B: now also IC9.2; no longer Q4.3, R10.1
- net OPT_MOT_PWR: now also IC7.2; no longer Q16.3, R34.1
- net OPT_SERVO1: now also IC10.12; no longer Q17.3, R36.1
- net OPT_SERVO2: now also IC10.10; no longer Q18.3, R38.1
- net OPT_SERVO3: now also IC10.8; no longer Q19.3, R40.1
- net OPT_SERVO4: now also IC10.2; no longer Q20.3, R42.1
- net OPT_SERVO5: now also IC11.12; no longer Q25.3, R52.1
- net OPT_SERVO6: now also IC11.10; no longer Q26.3, R54.1
- net OPT_SERVO7: now also IC11.8; no longer Q27.3, R56.1
- net OPT_SERVO8: now also IC11.2; no longer Q28.3, R58.1
- net OPT_SERVO_PWR: now also IC7.8; no longer Q15.3, R32.1
- net OPT_UART5_TX: now also IC7.12; no longer Q13.3, R28.1
- net SERVO_PWR: now also U$5.EN
- net UART5_RX: now also IC7.10; no longer Q14.3, R30.1
- net V+: now also C6.+, IC3.14, R23.1, R39.1, R55.1
- net V-: now also C6.-, IC3.7, J10.1
Routing:
- net GND: track 19.0 -> 548.8 mm, vias 0 -> 47
- net V-: track 0.00 -> 390.1 mm, vias 0 -> 42
- net V+: track 0.00 -> 337.5 mm, vias 0 -> 2
- net +12V_PWR: track 0.00 -> 272.3 mm, vias 0 -> 2
- net +5V: track 0.00 -> 267.4 mm, vias 0 -> 12
- net +3V3: track 0.00 -> 202.3 mm, vias 0 -> 4
- net STOP: track 0.00 -> 185.8 mm, vias 0 -> 4
- net +12V: track 0.00 -> 165.0 mm, vias 0 -> 1
- net OPT_MOT_PWR: track 0.00 -> 136.7 mm, vias 0 -> 8
- net SERVO_PWR: track 0.00 -> 99.5 mm, vias 0 -> 3
- net MOT_PWR: track 0.00 -> 98.5 mm, vias 0 -> 5
- net ENC_2A: track 0.00 -> 94.9 mm, vias 0 -> 8
- net ENC_3B: track 0.00 -> 93.4 mm, vias 0 -> 4
- net ENC_3A: track 0.00 -> 92.3 mm, vias 0 -> 3
- net TIRETTE: track 0.00 -> 82.3 mm
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- added copper zone on layer 1, net GND
- added copper zone on layer 16, net GND
- added copper zone on layer 1, net V-
- added copper zone on layer 16, net V-
Other:
- board text added: "6v"
- board text added: "Les Beffroyables Main board 0.1 by Hugo van Santen"
- board text added: "gnd"
- board text added: "sig"

Commit message: présentation schematics
Connections:
- net GND: now also OPT_MISC.9
- net STOP: now also Q5.4
Changed lines of the file:
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@@
 <wire x1="53.21714375" y1="79.5116375" x2="54.216478125" y2="78.512303125" width="0.4064" layer="1"/>
 <wire x1="48.26" y1="81.28" x2="50.0283625" y2="79.5116375" width="0.4064" layer="1"/>
+<contactref element="OPT_MISC" pad="9"/>
+<wire x1="96.84428125" y1="75.8621" x2="96.897634375" y2="77.62285625" width="0" layer="19" extent="1-1"/>
+<wire x1="96.52" y1="81.32" x2="96.897634375" y2="77.62285625" width="0" layer="19" extent="1-1"/>
+<wire x1="50.8" y1="90.17" x2="50.555896875" y2="89.594690625" width="0" layer="19" extent="1-1"/>
+<wire x1="17.78" y1="80.01" x2="17.75" y2="80.875" width="0" layer="19" extent="1-1"/>
+<wire x1="48.26" y1="87.63" x2="47.811253125" y2="86.850046875" width="0" layer="19" extent="1-1"/>
+<wire x1="58.57045" y1="78.512303125" x2="57.30045" y2="78.512303125" width="0" layer="19" extent="1-1"/>
+<wire x1="59.84045" y1="78.512303125" x2="58.57045" y2="78.512303125" width="0" layer="19" extent="1-1"/>
+<wire x1="73.57519375" y1="77.458846875" x2="74.5" y2="76.402309375" width="0" layer="19" extent="1-1"/>
+<wire x1="73.66" y1="74.93" x2="74.5" y2="76.25" width="0" layer="19" extent="1-1"/>
+<wire x1="77.806665625" y1="47.669409375" x2="75.955" y2="48.26" width="0" layer="19" extent="16-16"/>
+<wire x1="79.407659375" y1="47.733453125" x2="77.806665625" y2="47.669409375" width="0" layer="19" extent="1-1"/>
+<wire x1="68.58" y1="97.79" x2="66.44171875" y2="97.005" width="0" layer="19" extent="16-16"/>
+<wire x1="81.577496875" y1="77.95354375" x2="82.48104375" y2="80.207121875" width="0" layer="19" extent="1-1"/>
+<wire x1="79.998759375" y1="63.181621875" x2="79.998759375" y2="65.721621875" width="0" layer="19" extent="1-1"/>
+<wire x1="26.67" y1="92.71" x2="27.01" y2="90.17" width="0" layer="19" extent="1-1"/>
+<wire x1="88.51345" y1="76.6196375" x2="91.233484375" y2="76.033484375" width="0" layer="19" extent="16-16"/>
+<wire x1="86.69943125" y1="77.52669375" x2="88.51345" y2="76.6196375" width="0" layer="19" extent="1-1"/>
+<wire x1="46.99" y1="90.17" x2="48.26" y2="87.63" width="0" layer="19" extent="1-1"/>
+<wire x1="77.47" y1="72.39" x2="79.875" y2="70.875" width="0" layer="19" extent="1-1"/>
+<wire x1="67.945" y1="78.68" x2="68.72834375" y2="75.7907" width="0" layer="19" extent="1-1"/>
+<wire x1="97.007896875" y1="50.3116125" x2="99.118325" y2="48.103571875" width="0" layer="19" extent="1-1"/>
+<wire x1="93.475378125" y1="50.79174375" x2="97.007896875" y2="50.3116125" width="0" layer="19" extent="1-1"/>
+<wire x1="93.475378125" y1="52.06174375" x2="93.475378125" y2="50.79174375" width="0" layer="19" extent="1-1"/>
+<wire x1="93.475378125" y1="53.33174375" x2="93.475378125" y2="52.06174375" width="0" layer="19" extent="1-1"/>
+<wire x1="95.93458125" y1="54.45185" x2="93.475378125" y2="53.33174375" width="0" layer="19" extent="1-1"/>
+<wire x1="94.841246875" y1="57.980465625" x2="95.93458125" y2="54.45185" width="0" layer="19" extent="1-1"/>
+<wire x1="94.713165625" y1="61.054571875" x2="94.841246875" y2="57.980465625" width="0" layer="19" extent="1-1"/>
+<wire x1="11.43" y1="92.71" x2="11.43" y2="96.44296875" width="0" layer="19" extent="16-16"/>
+<wire x1="69.85" y1="93.98" x2="68.58" y2="97.79" width="0" layer="19" extent="1-1"/>
+<wire x1="22.86" y1="80.01" x2="19.05" y2="81.28" width="0" layer="19" extent="1-1"/>
+<wire x1="52.07" y1="83.65" x2="53.21714375" y2="79.5116375" width="0" layer="19" extent="1-1"/>
+<wire x1="31.75" y1="87.63" x2="27.94" y2="90.17" width="0" layer="19" extent="1-1"/>
+<wire x1="11.43" y1="77.47" x2="13.97" y2="81.28" width="0" layer="19" extent="1-1"/>
+<wire x1="7.62" y1="80.01" x2="11.43" y2="77.47" width="0" layer="19" extent="1-1"/>
+<wire x1="97.530915625" y1="71.10945" x2="96.84428125" y2="75.8621" width="0" layer="19" extent="1-1"/>
+<wire x1="17.78" y1="92.71" x2="15.24" y2="88.56" width="0" layer="19" extent="1-1"/>
+<wire x1="74.93" y1="93.98" x2="69.85" y2="93.98" width="0" layer="19" extent="1-1"/>
+<wire x1="74.93" y1="97.79" x2="74.93" y2="93.98" width="0" layer="19" extent="1-1"/>
+<wire x1="2.54" y1="80.01" x2="7.62" y2="80.01" width="0" layer="19" extent="1-1"/>
+<wire x1="38.1" y1="95.25" x2="39.363609375" y2="90.17" width="0" layer="19" extent="1-1"/>
+<wire x1="33.02" y1="95.25" x2="38.1" y2="95.25" width="0" layer="19" extent="1-1"/>
 </signal>
 <signal name="PAUSE_BUTTON">
@@
 <wire x1="15.24" y1="30.48" x2="38.1" y2="30.48" width="0.4064" layer="1"/>
 <wire x1="41.714890625" y1="30.48" x2="38.1" y2="30.48" width="0.4064" layer="16"/>
+<contactref element="Q5" pad="4"/>
+<wire x1="93.5" y1="49.625" x2="93.475378125" y2="49.52174375" width="0" layer="19" extent="1-1"/>
 </signal>
 <signal name="+4.1V">

Commit message: coorection board
modification board:
-correction alim découpage
-correction découpe contour
-correction ligne optocoupleur servo_enable
-correction ligne arduino imu
-amélioration connecteurs boutons
-ajout sortie 12v protégée (pour voltmètre)
ajout resistance 0ohm sur tous les composants 5V puissance (pour débug)
-ajout nomenclature sur board.
Parts:
- added J13: (no value), SparkFun-Connectors:1X08
- added J14: (no value), SparkFun-Connectors:MOLEX-1X2_LOCK
- added JP1: (no value), jumper:JP1
- added R10, R13, R14, R15, R16, R17, R6, R8: (no value), resistor:R0402
- J10: device SparkFun-Connectors:SCREWTERMINAL-3.5MM-8 -> SparkFun-Connectors:1X08
- moved J10 6.75 mm to (41.9, 27.0)
- moved IC4 1.27 mm to (38.1, 90.2)
- moved RN4 0.12 mm to (83.6, 61.3)
- moved OPT_MOT2 0.10 mm to (77.0, 54.6)
Connections:
- new net N$78: JP1.1, U$1.V+
- new net N$79: IC11.14, R6.2
- new net N$80: IC10.14, R8.2
- new net N$81: IC9.14, R10.2
- new net N$82: IC8.14, R13.2
- new net N$83: IC7.14, R14.2
- new net N$84: IC1.9, R15.2
- new net N$85: IC2.9, R16.2
- new net N$86: R17.2, U$2.VCC
- net +12V_PWR: now also J14.2
- net +3V3: now also R17.1; no longer U$2.VCC
- net +5V: now also R10.1, R13.1, R14.1, R15.1, R16.1, R6.1, R8.1; no longer IC1.9, IC10.14, IC11.14, IC2.9, IC7.14, IC8.14, IC9.14
- net GND: now also J14.1
- net I2C1_SCL: no longer U$2.SCL
- net I2C1_SDA: no longer U$2.SDA
- net I2C2_SCL: now also U$2.SCL
- net I2C2_SDA: now also U$2.SDA
- net MOT_1A: now also PCB1.P9.12; no longer PCB1.P9.28
- net OPT_SERVO_PWR: now also U$5.EN
- net SERVO_PWR: no longer U$5.EN
- net V+: now also JP1.2; no longer U$1.V+
- net V-: now also J13.1, J13.2, J13.3, J13.4, J13.5, J13.6, J13.7, J13.8
Routing:
- net OPT_SERVO_PWR: track 0.00 -> 121.8 mm, vias 0 -> 3
- net SERVO_PWR: track 99.5 -> 30.8 mm, vias 3 -> 1
- net V-: track 390.1 -> 358.4 mm, vias 42 -> 38
- net GND: track 548.8 -> 517.2 mm, vias 47 -> 46
- net MOT_1A: track 47.7 -> 71.2 mm
- net V+: track 337.5 -> 359.9 mm, vias 2 -> 4
- net +12V: track 165.0 -> 150.0 mm, vias 1 -> 2
- net I2C1_SCL: track 50.7 -> 62.9 mm
- net TIRETTE: track 82.3 -> 71.4 mm, vias 0 -> 1
- net STOP: track 185.8 -> 195.8 mm
- net ENC_3A: track 92.3 -> 99.6 mm, vias 3 -> 6
- net +5V: track 267.4 -> 274.1 mm, vias 12 -> 15
- net N$78: track 0.00 -> 5.61 mm
- net I2C2_SCL: track 45.0 -> 50.6 mm
- net I2C2_SDA: track 37.9 -> 42.0 mm
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Other:
- outline, holes or cut-outs redrawn
- board text added: "12V check"
- board text added: "arduino"
- board text added: "battery"
- board text added: "col1"
- board text added: "col2"
- board text added: "green"
- board text added: "i2c1"
- board text added: "i2c2"
- board text added: "orange"
- board text added: "red"
- board text added: "red button"
- board text added: "starter"
- board text added: "stop"
- board text added: "trigger"
- board text added: "uart1"
- board text added: "uart2"

Commit message: 2019 after eurobot
Parts:
- removed IC10, IC11, IC7, IC8, IC9: 74LS19D, 74xx-eu:SO14
- removed J10, J13: (no value), SparkFun-Connectors:1X08
- removed R10, R13, R14, R6, R8: (no value), resistor:R0402
- removed RN1: (no value), resistor-net:RN-8
- added J15, J16: (no value), SparkFun-Connectors:1X04
- added RN7: (no value), resistor-net:RN-5
- added U$3: LOGO, beffroyables:LOGO
- added U$6: LOGO_MAKERS, beffroyables:LOGO_MAKERS
- added X5, X6: (no value), con-phoenix-500:MSTBV2
- moved R25 18.1 mm to (69.2, 15.6), turned to 90 degrees
- moved R23 15.8 mm to (66.7, 15.6), turned to 90 degrees
- moved R19 14.8 mm to (61.6, 15.6), turned to 90 degrees
- moved R21 14.6 mm to (64.1, 15.6), turned to 90 degrees
- moved J14 13.3 mm to (44.5, 82.5)
- moved IC4 12.5 mm to (33.0, 78.7)
- moved OPT_MOT1 9.16 mm to (66.0, 22.9), turned to 90 degrees
- moved OPT_MOT2 8.16 mm to (85.1, 54.1), turned to 90 degrees
- moved OPT_MISC 6.75 mm to (83.5, 67.9), turned to 90 degrees
- moved R17 2.54 mm to (12.7, 12.7)
- moved U$2 2.54 mm to (34.3, 15.2)
Connections:
- removed net COL1: J10.5, PCB1.P8.4, RN1.5
- removed net N$19: IC9.1, OPT_MOT2.10, RN4.5
- removed net N$20: IC8.1, OPT_MOT1.10, RN3.5
- removed net N$21: IC8.9, OPT_MOT1.12, RN3.4
- removed net N$30: IC8.11, OPT_MOT1.14, RN3.3
- removed net N$31: IC8.13, OPT_MOT1.16, RN3.2
- removed net N$32: IC9.13, OPT_MOT2.16, RN4.2
- removed net N$33: IC9.11, OPT_MOT2.14, RN4.3
- removed net N$34: IC9.9, OPT_MOT2.12, RN4.4
- removed net N$35: IC10.1, OPT_SERVO1.10, RN6.5
- removed net N$36: IC10.9, OPT_SERVO1.12, RN6.4
- removed net N$37: IC10.11, OPT_SERVO1.14, RN6.3
- removed net N$4: IC7.13, OPT_MISC.16, RN2.2
- removed net N$46: IC10.13, OPT_SERVO1.16, RN6.2
- removed net N$47: IC11.13, OPT_SERVO2.16, RN5.2
- removed net N$48: IC11.11, OPT_SERVO2.14, RN5.3
- removed net N$49: IC11.9, OPT_SERVO2.12, RN5.4
- removed net N$50: IC11.1, OPT_SERVO2.10, RN5.5
- removed net N$53: IC7.11, OPT_MISC.14, RN2.3
- removed net N$62: IC7.9, OPT_MISC.12, RN2.4
- removed net N$63: IC7.1, OPT_MISC.10, RN2.5
- removed net N$79: IC11.14, R6.2
- removed net N$80: IC10.14, R8.2
- removed net N$81: IC9.14, R10.2
- removed net N$82: IC8.14, R13.2
- removed net N$83: IC7.14, R14.2
- removed net TIRETTE: J10.2, PCB1.P8.14, RN1.2
- new net INT_ACC: PCB1.P9.25, U$2.INT
- net +12V: now also J14.2
- net +12V_PWR: now also X5.1, X6.1; no longer J14.2
- net +3V3: now also R19.1, R21.1, R23.1, R25.1, R27.1, R29.1, R3.1, R31.1, R33.1, R35.1, R37.1, R39.1, R41.1, R5.1, R51.1, R53.1, R55.1, R57.1, R7.1, R9.1, RN7.1; no longer RN1.1
- net +5V: no longer R10.1, R13.1, R14.1, R6.1, R8.1
- net COL2: now also J16.1, PCB1.P9.23; no longer J10.4, RN1.4
- net GND: now also X5.2, X6.2; no longer IC10.7, IC11.7, IC7.7, IC8.7, IC9.7
- net GREEN: now also J16.4, RN7.2; no longer J10.8, RN1.8
- net MOT_PWR: now also PCB1.P8.31; no longer PCB1.P9.41
- net OPT_MOT1A: now also OPT_MOT1.16, RN3.2; no longer IC8.12
- net OPT_MOT1B: now also OPT_MOT1.14, RN3.3; no longer IC8.10
- net OPT_MOT2A: now also OPT_MOT1.12, RN3.4; no longer IC8.8
- net OPT_MOT2B: now also OPT_MOT1.10, RN3.5; no longer IC8.2
- net OPT_MOT3A: now also OPT_MOT2.16, RN4.2; no longer IC9.12
- net OPT_MOT3B: now also OPT_MOT2.14, RN4.3; no longer IC9.10
- net OPT_MOT4A: now also OPT_MOT2.12, RN4.4; no longer IC9.8
- net OPT_MOT4B: now also OPT_MOT2.10, RN4.5; no longer IC9.2
- net OPT_MOT_PWR: now also OPT_MISC.10, RN2.5; no longer IC7.2
- net OPT_SERVO1: now also OPT_SERVO1.16, RN6.2; no longer IC10.12
- net OPT_SERVO2: now also OPT_SERVO1.14, RN6.3; no longer IC10.10
- net OPT_SERVO3: now also OPT_SERVO1.12, RN6.4; no longer IC10.8
- net OPT_SERVO4: now also OPT_SERVO1.10, RN6.5; no longer IC10.2
- net OPT_SERVO5: now also OPT_SERVO2.16, RN5.2; no longer IC11.12
- net OPT_SERVO6: now also OPT_SERVO2.14, RN5.3; no longer IC11.10
- net OPT_SERVO7: now also OPT_SERVO2.12, RN5.4; no longer IC11.8
- net OPT_SERVO8: now also OPT_SERVO2.10, RN5.5; no longer IC11.2
- net OPT_SERVO_PWR: now also OPT_MISC.12, RN2.4; no longer IC7.8
- net OPT_UART5_TX: now also OPT_MISC.16, RN2.2; no longer IC7.12
- net ORANGE: now also J16.3, RN7.3; no longer J10.7, RN1.7
- net RED: now also J16.2, PCB1.P8.32, RN7.4; no longer J10.6, PCB1.P8.6, RN1.6
- net STOP: no longer J10.3, RN1.3
- net UART5_RX: now also OPT_MISC.14, RN2.3; no longer IC7.10
- net V+: no longer R19.1, R21.1, R23.1, R25.1, R27.1, R29.1, R3.1, R31.1, R33.1, R35.1, R37.1, R39.1, R41.1, R5.1, R51.1, R53.1, R55.1, R57.1, R7.1, R9.1
- net V-: now also J15.1, J15.2, J15.3, J15.4; no longer J10.1, J13.1, J13.2, J13.3, J13.4, J13.5, J13.6, J13.7, J13.8
Routing:
- net V+: track 359.9 -> 148.7 mm, vias 4 -> 1
- net +3V3: track 206.3 -> 406.9 mm, vias 5 -> 10
- net GND: track 517.2 -> 440.2 mm, vias 46 -> 36
- net TIRETTE: track 71.4 -> 0.00 mm, vias 1 -> 0
- net N$14: track 3.97 -> 53.3 mm, vias 0 -> 2
- net COL1: track 48.6 -> 0.00 mm
- net COL2: track 46.6 -> 88.0 mm, vias 0 -> 3
- net STOP: track 195.8 -> 157.4 mm
- net N$13: track 3.78 -> 35.2 mm, vias 0 -> 4
- net INT_ACC: track 0.00 -> 28.8 mm, vias 0 -> 2
- net N$19: track 26.4 -> 0.00 mm
- net OPT_MOT2A: track 12.7 -> 36.9 mm
- net N$31: track 22.6 -> 0.00 mm
- net N$21: track 21.4 -> 0.00 mm, vias 1 -> 0
- net N$69: track 2.18 -> 23.3 mm
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Other:
- outline, holes or cut-outs redrawn
- board text added: "Les Beffroyables Main board 0.2b by Hugo van Santen"
- board text removed: "Les Beffroyables Main board 0.1 by Hugo van Santen"
