File: asserv_shield/shield/motor_shield.sch (EAGLE design)
At the start: 83 parts, among them IC1 L298, IC2 L298

Commit message: PCB v0.1
Parts:
- removed Q1, Q10, Q11, Q12, Q13, Q14, Q15, Q16, Q17, Q18, Q19, Q2, Q20, Q25, Q26, Q27, Q28, Q3, Q4, Q9: (no value), semicon-smd-ipc:NPN-TRANSISTOR_SOT23
- removed R10, R20, R22, R24, R26, R28, R30, R32, R34, R36, R38, R40, R42, R52, R54, R56, R58, R6, R8: 800, rcl:R-EU_M0805
- added C1: (no value), BeagleBone_Blue:SPARKFUN-CAPACITORS_CAP0805
- added C2, C3, C4, C5, C6: (no value), BeagleBone_Blue:CPOL-US140CLH-1010
- added IC10, IC11, IC7, IC8, IC9: 74LS19D, 74xx-eu:74LS19D
- added IC3: 4030D, 40xx:4030D
- added IC4: 7805DT, linear:7805DT
- added IC5: MAX6520, maxim:MAX6520
- added IC6: LM358D, linear:LM358D
- added J10: (no value), SparkFun-Connectors:CONN_083.5MM-8
- added J11: (no value), con-jack:JACK-PLUG1
- added J12: (no value), SparkFun-Connectors:CONN_02POLAR_LOCK
- added K1: RT33K012, relay:RT33K012
- added Q5, Q6: STRAWSON_EAGLE_LIB_MOSFET-NCHANNEL, BeagleBone_Blue:STRAWSON_EAGLE_LIB_MOSFET-NCHANNEL
- added R11: 6k, rcl:R-EU_M0805
- added R12: 3k, rcl:R-EU_M0805
- added RN1: (no value), resistor-net:RNX7
- added RN2, RN3, RN4, RN5, RN6: 680, resistor-net:RN04
- added U$5: XL6009, beffroyables:XL6009
- added X2, X3: (no value), con-phoenix-500:MSTBV2
- R4: value 800 -> 6k
Connections:
- removed net EN2A: PCB1.P8.35
- removed net MOT_DIR1A: PCB1.P9.28
- removed net MOT_PMW_1B: PCB1.P9.16
- new net +12V_PWR: C2.+, C3.+, C4.+, C5.+, IC1.VS, IC2.VS, J11.3, U$5.IN+, X1-2.SK
- new net +4.1V: U$4.PWR, U$5.OUT+
- new net COL1: J10.5, PCB1.P8.4, RN1-4.1
- new net COL2: J10.4, PCB1.P8.5, RN1-3.1
- new net DOOR_MOT_1A: IC3A.O, OPT_MOT1A.C
- new net DOOR_MOT_2A: IC3B.O, OPT_MOT1C.C
- new net DOOR_MOT_3A: IC3C.O, OPT_MOT2A.C
- new net DOOR_MOT_4A: IC3D.O, OPT_MOT2C.C
- new net GREEN: J10.8, PCB1.P8.8, RN1-7.1
- new net MOT_PWM_1B: IC3B.I0, PCB1.P9.16
- new net N$64: IC5.OUT, IC6A.-IN
- new net N$73: IC6A.OUT, R4.2
- new net N$74: K12.SA, K12.SB, X2-2.SK, X3-1.SK
- new net N$75: K11.1, Q6.S
- new net N$76: IC6A.+IN, J12.2, R11.1, R12.2
- new net N$77: C1.1, Q6.G, R4.1
- new net ORANGE: J10.7, PCB1.P8.7, RN1-6.1
- new net RED: J10.6, PCB1.P8.6, RN1-5.1
- new net STOP: J10.3, PCB1.P8.3, Q5.G, RN1-2.1
- new net TIRETTE: J10.2, PCB1.P8.14, RN1-1.1
- net +12V: now also IC4.VI, K11.2, K12.PA, K12.PB, R11.2, X1-1.SK, X2-1.SK; no longer IC1.VS, IC2.VS, X1-2.SK
- net +3V3: now also RN1_.1
- net +5V: now also IC1.VCC, IC10P.VCC, IC11P.VCC, IC2.VCC, IC4.VO, IC5.IN, IC6P.V+, IC7P.VCC, IC8P.VCC, IC9P.VCC, RN2.1, RN3.1, RN4.1, RN5.1, RN6.1; no longer R10.2, R20.2, R22.2, R24.2, R26.2, R28.2, R30.2, R32.2, R34.2, R36.2, R38.2, R4.2, R40.2, R42.2, R52.2, R54.2, R56.2, R58.2, R6.2, R8.2
- net ENC_2A: now also PCB1.P8.35
- net GND: now also C1.2, C2.-, C3.-, C4.-, C5.-, IC10P.GND, IC11P.GND, IC4.GND, IC5.GND, IC6P.V-, IC7P.GND, IC8P.GND, IC9P.GND, J12.1, Q5.D, Q6.D, R12.1, U$5.IN-, U$5.OUT-, X3-2.SK; no longer OPT_MISCD.EMIT, Q1.E, Q10.E, Q11.E, Q12.E, Q13.E, Q14.E, Q15.E, Q16.E, Q17.E, Q18.E, Q19.E, Q2.E, Q20.E, Q25.E, Q26.E, Q27.E, Q28.E, Q3.E, Q4.E, Q9.E, X1-1.SK
- net I2C2_SCL: no longer J9.1
- net I2C2_SDA: now also J9.1
- net MOT_1A: now also IC3A.I1, PCB1.P9.28; no longer OPT_MOT1A.C
- net MOT_2A: now also IC3B.I1; no longer OPT_MOT1C.C
- net MOT_3A: now also IC3C.I1; no longer OPT_MOT2A.C
- net MOT_4A: now also IC3D.I1; no longer OPT_MOT2C.C
- net MOT_PWM_1A: now also IC3A.I0
- net MOT_PWM_2A: now also IC3C.I0
- net MOT_PWM_2B: now also IC3D.I0
- net N$10: now also J11.1, Q5.S; no longer U$4.PWR
- net N$19: now also IC9D.I, RN4.5; no longer Q4.B
- net N$20: now also IC8D.I, RN3.5; no longer Q12.B
- net N$21: now also IC8C.I, RN3.4; no longer Q11.B
- net N$30: now also IC8B.I, RN3.3; no longer Q10.B
- net N$31: now also IC8A.I, RN3.2; no longer Q9.B
- net N$32: now also IC9A.I, RN4.2; no longer Q1.B
- net N$33: now also IC9B.I, RN4.3; no longer Q2.B
- net N$34: now also IC9C.I, RN4.4; no longer Q3.B
- net N$35: now also IC10D.I, RN6.5; no longer Q20.B
- net N$36: now also IC10C.I, RN6.4; no longer Q19.B
- net N$37: now also IC10B.I, RN6.3; no longer Q18.B
- net N$4: now also IC7A.I, RN2.2; no longer Q13.B
- net N$46: now also IC10A.I, RN6.2; no longer Q17.B
- net N$47: now also IC11A.I, RN5.2; no longer Q25.B
- net N$48: now also IC11B.I, RN5.3; no longer Q26.B
- net N$49: now also IC11C.I, RN5.4; no longer Q27.B
- net N$50: now also IC11D.I, RN5.5; no longer Q28.B
- net N$53: now also IC7B.I, RN2.3; no longer Q14.B
- net N$62: now also IC7C.I, RN2.4; no longer Q15.B
- net N$63: now also IC7D.I, RN2.5; no longer Q16.B
- net OPT_MOT1A: now also IC8A.O; no longer Q9.C, R20.1
- net OPT_MOT1B: now also IC8B.O; no longer Q10.C, R22.1
- net OPT_MOT2A: now also IC8C.O; no longer Q11.C, R24.1
- net OPT_MOT2B: now also IC8D.O; no longer Q12.C, R26.1
- net OPT_MOT3A: now also IC9A.O; no longer Q1.C, R4.1
- net OPT_MOT3B: now also IC9B.O; no longer Q2.C, R6.1
- net OPT_MOT4A: now also IC9C.O; no longer Q3.C, R8.1
- net OPT_MOT4B: now also IC9D.O; no longer Q4.C, R10.1
- net OPT_MOT_PWR: now also IC7D.O; no longer Q16.C, R34.1
- net OPT_SERVO1: now also IC10A.O; no longer Q17.C, R36.1
- net OPT_SERVO2: now also IC10B.O; no longer Q18.C, R38.1
- net OPT_SERVO3: now also IC10C.O; no longer Q19.C, R40.1
- net OPT_SERVO4: now also IC10D.O; no longer Q20.C, R42.1
- net OPT_SERVO5: now also IC11A.O; no longer Q25.C, R52.1
- net OPT_SERVO6: now also IC11B.O; no longer Q26.C, R54.1
- net OPT_SERVO7: now also IC11C.O; no longer Q27.C, R56.1
- net OPT_SERVO8: now also IC11D.O; no longer Q28.C, R58.1
- net OPT_SERVO_PWR: now also IC7C.O; no longer Q15.C, R32.1
- net OPT_UART5_TX: now also IC7A.O; no longer Q13.C, R28.1
- net SERVO_PWR: now also U$5.EN
- net UART5_RX: now also IC7B.O; no longer Q14.C, R30.1
- net V+: now also C6.+, IC3P.VDD, R23.1, R39.1, R55.1
- net V-: now also C6.-, IC3P.VSS, J10.1
Other:
- moved on the sheet: R23, R39, R4, R55, R7, X1-1, X1-2

Commit message: minor updates
Connections:
- net GND: now also Q5.S, Q6.S; no longer Q5.D, Q6.D
- net N$10: now also Q5.D; no longer Q5.S
- net N$75: now also Q6.D; no longer Q6.S
- net STOP: no longer Q5.G
Other:
- moved on the sheet: Q5, Q6
Changed lines of the file:
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@@
 <instance part="SUPPLY2" gate="P" x="160.02" y="-114.3"/>
 <instance part="J11" gate="G$1" x="381" y="-93.98" rot="R180"/>
-<instance part="P+49" gate="1" x="365.76" y="-93.98"/>
-<instance part="Q5" gate="G$1" x="350.52" y="-91.44" rot="R90"/>
-<instance part="GND25" gate="1" x="345.44" y="-93.98"/>
+<instance part="P+49" gate="1" x="368.3" y="-93.98"/>
+<instance part="Q5" gate="G$1" x="350.52" y="-96.52" rot="R270"/>
+<instance part="GND25" gate="1" x="340.36" y="-99.06"/>
 <instance part="P+50" gate="1" x="279.4" y="-27.94"/>
 <instance part="P+51" gate="1" x="198.12" y="-27.94"/>
@@
 <instance part="X2" gate="-1" x="121.92" y="187.96" rot="R270"/>
 <instance part="X2" gate="-2" x="116.84" y="187.96" rot="R270"/>
-<instance part="Q6" gate="G$1" x="111.76" y="154.94" rot="R90"/>
+<instance part="Q6" gate="G$1" x="111.76" y="154.94" rot="R270"/>
 <instance part="IC5" gate="-1" x="160.02" y="149.86" rot="R180"/>
 <instance part="P+2" gate="1" x="167.64" y="149.86"/>
@@
 </segment>
 <segment>
-<pinref part="Q5" gate="G$1" pin="D"/>
-<pinref part="GND25" gate="1" pin="GND"/>
-</segment>
-<segment>
-<pinref part="Q6" gate="G$1" pin="D"/>
 <pinref part="GND4" gate="1" pin="GND"/>
-<wire x1="104.14" y1="154.94" x2="106.68" y2="154.94" width="0.1524" layer="91"/>
 <pinref part="X3" gate="-2" pin="SK"/>
 <wire x1="101.6" y1="165.1" x2="101.6" y2="154.94" width="0.1524" layer="91"/>
 <wire x1="101.6" y1="154.94" x2="104.14" y2="154.94" width="0.1524" layer="91"/>
+<wire x1="104.14" y1="154.94" x2="106.68" y2="154.94" width="0.1524" layer="91"/>
+<pinref part="Q6" gate="G$1" pin="S"/>
 </segment>
 <segment>
@@
 <wire x1="-30.48" y1="-99.06" x2="-30.48" y2="-104.14" width="0.1524" layer="91"/>
 <pinref part="GND43" gate="1" pin="GND"/>
+</segment>
+<segment>
+<pinref part="GND25" gate="1" pin="GND"/>
+<pinref part="Q5" gate="G$1" pin="S"/>
+<wire x1="345.44" y1="-96.52" x2="340.36" y2="-96.52" width="0.1524" layer="91"/>
 </segment>
 </net>
@@
 </segment>
 <segment>
-<pinref part="Q5" gate="G$1" pin="G"/>
-<wire x1="350.52" y1="-99.06" x2="350.52" y2="-101.6" width="0.1524" layer="91"/>
-<label x="347.98" y="-104.14" size="1.778" layer="95"/>
+<label x="342.9" y="-86.36" size="1.778" layer="95"/>
+<wire x1="350.52" y1="-86.36" x2="350.52" y2="-88.9" width="0.1524" layer="91"/>
 </segment>
 <segment>
@@
 <wire x1="160.02" y1="-116.84" x2="157.48" y2="-116.84" width="0.1524" layer="91"/>
 <pinref part="SUPPLY2" gate="P" pin="+4.1V"/>
-</segment>
-</net>
-<net name="N$10" class="0">
-<segment>
-<pinref part="Q5" gate="G$1" pin="S"/>
-<pinref part="J11" gate="G$1" pin="1"/>
-<wire x1="355.6" y1="-91.44" x2="375.92" y2="-91.44" width="0.1524" layer="91"/>
 </segment>
 </net>
@@
 <segment>
 <pinref part="K1" gate="1" pin="1"/>
-<wire x1="116.84" y1="154.94" x2="121.92" y2="154.94" width="0.1524" layer="91"/>
-<pinref part="Q6" gate="G$1" pin="S"/>
+<wire x1="121.92" y1="154.94" x2="116.84" y2="154.94" width="0.1524" layer="91"/>
+<pinref part="Q6" gate="G$1" pin="D"/>
 </segment>
 </net>
@@
 <pinref part="J11" gate="G$1" pin="3"/>
 <pinref part="P+49" gate="1" pin="+12V"/>
-<wire x1="375.92" y1="-96.52" x2="365.76" y2="-96.52" width="0.1524" layer="91"/>
 <label x="363.22" y="-101.6" size="1.778" layer="95"/>
+<wire x1="368.3" y1="-96.52" x2="375.92" y2="-96.52" width="0.1524" layer="91"/>
 </segment>
 <segment>
@@
 <net name="N$77" class="0">
 <segment>
-<pinref part="Q6" gate="G$1" pin="G"/>
 <pinref part="R4" gate="G$1" pin="1"/>
-<wire x1="111.76" y1="147.32" x2="116.84" y2="147.32" width="0.1524" layer="91"/>
 <pinref part="C1" gate="G$1" pin="1"/>
 <wire x1="116.84" y1="147.32" x2="124.46" y2="147.32" width="0.1524" layer="91"/>
 <junction x="116.84" y="147.32"/>
+<wire x1="116.84" y1="147.32" x2="96.52" y2="147.32" width="0.1524" layer="91"/>
+<wire x1="96.52" y1="147.32" x2="96.52" y2="162.56" width="0.1524" layer="91"/>
+<pinref part="Q6" gate="G$1" pin="G"/>
+<wire x1="96.52" y1="162.56" x2="111.76" y2="162.56" width="0.1524" layer="91"/>
 </segment>
 </net>
@@
 </segment>
 </net>
+<net name="N$10" class="0">
+<segment>
+<pinref part="Q5" gate="G$1" pin="D"/>
+<wire x1="355.6" y1="-96.52" x2="355.6" y2="-91.44" width="0.1524" layer="91"/>
+<pinref part="J11" gate="G$1" pin="1"/>
+<wire x1="355.6" y1="-91.44" x2="375.92" y2="-91.44" width="0.1524" layer="91"/>
+</segment>
+</net>

Commit message: présentation schematics
Connections:
- net GND: now also OPT_MISCD.EMIT
- net STOP: now also Q5.G
Other:
- note added: "Par Hugo van Santen Pour les Beffroyables"
- note added: "alimentation"
- note added: "connceteurs et contrôle puissance"
- note added: "connecteur alime+ gestion batterie"
- note added: "isolation"
- note added: "shield+motor control logic"
- moved on the sheet: C1, C2, C3, C4, C5, C6, IC1, IC10A, IC10B, IC10C, IC10D, IC10P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

Commit message: coorection board
modification board:
-correction alim découpage
-correction découpe contour
-correction ligne optocoupleur servo_enable
-correction ligne arduino imu
-amélioration connecteurs boutons
-ajout sortie 12v protégée (pour voltmètre)
ajout resistance 0ohm sur tous les composants 5V puissance (pour débug)
-ajout nomenclature sur board.
Parts:
- added J13: (no value), SparkFun-Connectors:CONN_08"
- added J14: (no value), SparkFun-Connectors:CONN_02POLAR_LOCK
- added JP1: (no value), jumper:JP1E
- added R10, R13, R14, R15, R16, R17, R6, R8: (no value), resistor:R-EU_R0402
- J10: device SparkFun-Connectors:CONN_083.5MM-8 -> SparkFun-Connectors:CONN_08"
Connections:
- new net N$78: JP1.1, U$1.V+
- new net N$79: IC11P.VCC, R6.2
- new net N$80: IC10P.VCC, R8.2
- new net N$81: IC9P.VCC, R10.2
- new net N$82: IC8P.VCC, R13.2
- new net N$83: IC7P.VCC, R14.2
- new net N$84: IC1.VCC, R15.2
- new net N$85: IC2.VCC, R16.2
- new net N$86: R17.2, U$2.VCC
- net +12V_PWR: now also J14.2
- net +3V3: now also R17.1; no longer U$2.VCC
- net +5V: now also R10.1, R13.1, R14.1, R15.1, R16.1, R6.1, R8.1; no longer IC1.VCC, IC10P.VCC, IC11P.VCC, IC2.VCC, IC7P.VCC, IC8P.VCC, IC9P.VCC
- net GND: now also J14.1
- net I2C1_SCL: no longer U$2.SCL
- net I2C1_SDA: no longer U$2.SDA
- net I2C2_SCL: now also U$2.SCL
- net I2C2_SDA: now also U$2.SDA
- net MOT_1A: now also PCB1.P9.12; no longer PCB1.P9.28
- net OPT_SERVO_PWR: now also U$5.EN
- net SERVO_PWR: no longer U$5.EN
- net V+: now also JP1.2; no longer U$1.V+
- net V-: now also J13.1, J13.2, J13.3, J13.4, J13.5, J13.6, J13.7, J13.8
Other:
- moved on the sheet: R53

Commit message: 2019 after eurobot
Parts:
- removed IC10, IC11, IC7, IC8, IC9: 74LS19D, 74xx-eu:74LS19D
- removed J10, J13: (no value), SparkFun-Connectors:CONN_08"
- removed R10, R13, R14, R6, R8: (no value), resistor:R-EU_R0402
- removed RN1: (no value), resistor-net:RNX7
- added J15, J16: (no value), SparkFun-Connectors:CONN_04
- added RN7: (no value), resistor-net:RN04
- added U$3: LOGO, beffroyables:LOGO
- added U$6: LOGO_MAKERS, beffroyables:LOGO_MAKERS
- added X5, X6: (no value), con-phoenix-500:MSTBV2
Connections:
- removed net COL1: J10.5, PCB1.P8.4, RN1-4.1
- removed net N$19: IC9D.I, OPT_MOT2D.COL, RN4.5
- removed net N$20: IC8D.I, OPT_MOT1D.COL, RN3.5
- removed net N$21: IC8C.I, OPT_MOT1C.COL, RN3.4
- removed net N$30: IC8B.I, OPT_MOT1B.COL, RN3.3
- removed net N$31: IC8A.I, OPT_MOT1A.COL, RN3.2
- removed net N$32: IC9A.I, OPT_MOT2A.COL, RN4.2
- removed net N$33: IC9B.I, OPT_MOT2B.COL, RN4.3
- removed net N$34: IC9C.I, OPT_MOT2C.COL, RN4.4
- removed net N$35: IC10D.I, OPT_SERVO1D.COL, RN6.5
- removed net N$36: IC10C.I, OPT_SERVO1C.COL, RN6.4
- removed net N$37: IC10B.I, OPT_SERVO1B.COL, RN6.3
- removed net N$4: IC7A.I, OPT_MISCA.COL, RN2.2
- removed net N$46: IC10A.I, OPT_SERVO1A.COL, RN6.2
- removed net N$47: IC11A.I, OPT_SERVO2A.COL, RN5.2
- removed net N$48: IC11B.I, OPT_SERVO2B.COL, RN5.3
- removed net N$49: IC11C.I, OPT_SERVO2C.COL, RN5.4
- removed net N$50: IC11D.I, OPT_SERVO2D.COL, RN5.5
- removed net N$53: IC7B.I, OPT_MISCB.COL, RN2.3
- removed net N$62: IC7C.I, OPT_MISCC.COL, RN2.4
- removed net N$63: IC7D.I, OPT_MISCD.COL, RN2.5
- removed net N$79: IC11P.VCC, R6.2
- removed net N$80: IC10P.VCC, R8.2
- removed net N$81: IC9P.VCC, R10.2
- removed net N$82: IC8P.VCC, R13.2
- removed net N$83: IC7P.VCC, R14.2
- removed net TIRETTE: J10.2, PCB1.P8.14, RN1-1.1
- new net INT_ACC: PCB1.P9.25, U$2.INT
- net +12V: now also J14.2
- net +12V_PWR: now also X5-1.SK, X6-1.SK; no longer J14.2
- net +3V3: now also R19.1, R21.1, R23.1, R25.1, R27.1, R29.1, R3.1, R31.1, R33.1, R35.1, R37.1, R39.1, R41.1, R5.1, R51.1, R53.1, R55.1, R57.1, R7.1, R9.1, RN7.1; no longer RN1_.1
- net +5V: no longer R10.1, R13.1, R14.1, R6.1, R8.1
- net COL2: now also J16.1, PCB1.P9.23; no longer J10.4, RN1-3.1
- net GND: now also X5-2.SK, X6-2.SK; no longer IC10P.GND, IC11P.GND, IC7P.GND, IC8P.GND, IC9P.GND
- net GREEN: now also J16.4, RN7.2; no longer J10.8, RN1-7.1
- net MOT_PWR: now also PCB1.P8.31; no longer PCB1.P9.41
- net OPT_MOT1A: now also OPT_MOT1A.COL, RN3.2; no longer IC8A.O
- net OPT_MOT1B: now also OPT_MOT1B.COL, RN3.3; no longer IC8B.O
- net OPT_MOT2A: now also OPT_MOT1C.COL, RN3.4; no longer IC8C.O
- net OPT_MOT2B: now also OPT_MOT1D.COL, RN3.5; no longer IC8D.O
- net OPT_MOT3A: now also OPT_MOT2A.COL, RN4.2; no longer IC9A.O
- net OPT_MOT3B: now also OPT_MOT2B.COL, RN4.3; no longer IC9B.O
- net OPT_MOT4A: now also OPT_MOT2C.COL, RN4.4; no longer IC9C.O
- net OPT_MOT4B: now also OPT_MOT2D.COL, RN4.5; no longer IC9D.O
- net OPT_MOT_PWR: now also OPT_MISCD.COL, RN2.5; no longer IC7D.O
- net OPT_SERVO1: now also OPT_SERVO1A.COL, RN6.2; no longer IC10A.O
- net OPT_SERVO2: now also OPT_SERVO1B.COL, RN6.3; no longer IC10B.O
- net OPT_SERVO3: now also OPT_SERVO1C.COL, RN6.4; no longer IC10C.O
- net OPT_SERVO4: now also OPT_SERVO1D.COL, RN6.5; no longer IC10D.O
- net OPT_SERVO5: now also OPT_SERVO2A.COL, RN5.2; no longer IC11A.O
- net OPT_SERVO6: now also OPT_SERVO2B.COL, RN5.3; no longer IC11B.O
- net OPT_SERVO7: now also OPT_SERVO2C.COL, RN5.4; no longer IC11C.O
- net OPT_SERVO8: now also OPT_SERVO2D.COL, RN5.5; no longer IC11D.O
- net OPT_SERVO_PWR: now also OPT_MISCC.COL, RN2.4; no longer IC7C.O
- net OPT_UART5_TX: now also OPT_MISCA.COL, RN2.2; no longer IC7A.O
- net ORANGE: now also J16.3, RN7.3; no longer J10.7, RN1-6.1
- net RED: now also J16.2, PCB1.P8.32, RN7.4; no longer J10.6, PCB1.P8.6, RN1-5.1
- net STOP: no longer J10.3, RN1-2.1
- net UART5_RX: now also OPT_MISCB.COL, RN2.3; no longer IC7B.O
- net V+: no longer R19.1, R21.1, R23.1, R25.1, R27.1, R29.1, R3.1, R31.1, R33.1, R35.1, R37.1, R39.1, R41.1, R5.1, R51.1, R53.1, R55.1, R57.1, R7.1, R9.1
- net V-: now also J15.1, J15.2, J15.3, J15.4; no longer J10.1, J13.1, J13.2, J13.3, J13.4, J13.5, J13.6, J13.7, J13.8
